File: Medidor_lata/Medidor_lata.sch (KiCad schematic (older format))
At the start: 7 parts, among them J1 Conn_01x02_Female, SW1 SW_Push, U1 ATmega328P-AU, Y1 Crystal

Commit message: Hemos trabajado en nueva version de sistema de medicio
Parts:
- removed SW1: SW_Push, Button_Switch_THT:Push_E-Switch_KS01Q01, symbol Switch:SW_Push
- added D1, D2: LED, LED_THT:LED_D3.0mm, symbol Device:LED
- added Q1, Q3: BC847, Package_TO_SOT_SMD:SOT-23, symbol Transistor_BJT:BC847
- added Q2: BC856, Package_TO_SOT_SMD:SOT-23, symbol Transistor_BJT:BC856
- added R2, R3, R4, R5, R6, R7, R8: R, Resistor_SMD:R_0805_2012Metric, symbol Device:R
- added Sw1, Sw2, Sw3, Sw4: Pulsador, Button_Switch_Keyboard:Pulsador, symbol Switch:Pulsador
- added U2: PC817, Package_DIP:DIP-4_W7.62mm, symbol Isolator:PC817
- C1, C2: footprint Capacitor_THT:C_Axial_L3.8mm_D2.6mm_P7.50mm_Horizontal -> Capacitor_SMD:C_0805_2012Metric
- J1: footprint Connector_Hirose:Hirose_DF13-02P-1.25DS_1x02_P1.25mm_Horizontal -> Connector_JST:JST_EH_B02B-EH-A_1x02_P2.50mm_Vertical
- R1: footprint Resistor_THT:R_Axial_DIN0204_L3.6mm_D1.6mm_P5.08mm_Horizontal -> Resistor_SMD:R_0805_2012Metric
Connections:
- wire segments 28 -> 88
- no-connect marks 24 -> 19
