File: Medidor_lata/Lector infrarojo/lector infrarojo/lector infrarojo.sch (KiCad schematic (older format))
At the start: 16 parts, among them J1 Conn_01x02_Female, J2 Conn_01x02_Female

Commit message: Cambios de medidor
Parts:
- added Q1, Q2, Q3, Q4, Q5, Q6, Q7: BC857, Package_TO_SOT_SMD:SOT-23, symbol Transistor_BJT:BC857
- added R10, R11, R12, R13, R14, R15, R16, R17, R18, R19, R20, R21, R8, R9: R, Resistor_SMD:R_0805_2012Metric, symbol Device:R
Connections:
- wire segments 68 -> 140
