File: Medidor_lata/Medidor_V1.2/Medidor_V1.2.kicad_pcb (KiCad board)
At the start: 2 copper layers, 90 x 90 mm, 13 parts, among them J1 Conn_01x02_Female, Sw1 Pulsador, U1 CC56-12EWA, U2 ATmega328-AU

Commit message: Cambios de medidor
Parts:
- added J2: Conn_01x04_Female, Connector_JST:JST_EH_B04B-EH-A_1x04_P2.50mm_Vertical, B.Cu at (169.4, 76.7)
- moved Sw1 39.4 mm to (174.7, 57.0), turned to 180 degrees
- moved J1 22.6 mm to (103.7, 66.3), turned to 90 degrees
- moved U2 12.2 mm to (130.2, 63.5)
Connections:
- U2 pad 16: Net-(U2-Pad16) -> Net-(R1-Pad2)
- U2 pad 17: Net-(U2-Pad17) -> Net-(R2-Pad2)
- U2 pad 30: Net-(R1-Pad2) -> Net-(J2-Pad3)
- U2 pad 31: Net-(R2-Pad2) -> Net-(J2-Pad4)
