File: Medidor_lata/Medidor_V1.2/Medidor_V1.2.sch (KiCad schematic (older format))
At the start: 13 parts, among them J1 Conn_01x02_Female, Sw1 Pulsador, U1 CC56-12EWA, U2 ATmega328-AU

Commit message: Cambios de medidor
Parts:
- added J2: Conn_01x04_Female, Connector_JST:JST_EH_B04B-EH-A_1x04_P2.50mm_Vertical, symbol Connector:Conn_01x04_Female
Connections:
- wire segments 84 -> 100
- no-connect marks 14 -> 12
Changed lines of the file:
@@
 	3950 3200 4350 3200
 Wire Wire Line
-	3350 4550 3900 4550
-Wire Wire Line
-	3900 4550 3900 2900
-Wire Wire Line
 	3900 2900 4350 2900
-Wire Wire Line
-	4350 2600 3850 2600
-Wire Wire Line
-	3850 2600 3850 4450
-Wire Wire Line
-	3850 4450 3350 4450
 Wire Wire Line
 	7400 3000 7400 2200
@@
 $EndComp
 NoConn ~ 2850 2450
-NoConn ~ 3350 3150
-NoConn ~ 3350 3250
 NoConn ~ 3350 3350
 NoConn ~ 3350 3450
@@
 Wire Wire Line
 	1550 5700 2750 5700
+Wire Wire Line
+	3900 3250 3350 3250
+Wire Wire Line
+	3900 2900 3900 3250
+Wire Wire Line
+	3350 3150 3450 3150
+Wire Wire Line
+	3450 3150 3500 3100
+Wire Wire Line
+	3500 3100 3800 3100
+Wire Wire Line
+	3800 3100 3800 2600
+Wire Wire Line
+	3800 2600 4350 2600
+$Comp
+L Connector:Conn_01x04_Female J2
+U 1 1 5BBD60F2
+P 2000 3700
+F 0 "J2" H 2027 3676 50  0000 L CNN
+F 1 "Conn_01x04_Female" H 2027 3585 50  0000 L CNN
+F 2 "Connector_JST:JST_EH_B04B-EH-A_1x04_P2.50mm_Vertical" H 2000 3700 50  0001 C CNN
+F 3 "~" H 2000 3700 50  0001 C CNN
+	1    2000 3700
+	1    0    0    -1
+$EndComp
+Wire Wire Line
+	1800 3600 1800 3200
+Wire Wire Line
+	1800 3200 1550 3200
+Connection ~ 1550 3200
+Wire Wire Line
+	1800 3700 1700 3700
+Wire Wire Line
+	1700 3700 1700 3300
+Wire Wire Line
+	1700 3300 1550 3300
+Connection ~ 1550 3300
+Wire Wire Line
+	1800 3800 1650 3800
+Wire Wire Line
+	1650 3800 1650 5500
+Wire Wire Line
+	1650 5500 3800 5500
+Wire Wire Line
+	3800 4450 3350 4450
+Wire Wire Line
+	3800 4450 3800 5500
+Wire Wire Line
+	1800 3900 1800 5550
+Wire Wire Line
+	1800 5550 3900 5550
+Wire Wire Line
+	3900 5550 3900 4550
+Wire Wire Line
+	3900 4550 3350 4550
 $EndSCHEMATC
