File: Medidor_lata/ArduprofeVEJCP/ArduprofeVEJCP.kicad_pcb (KiCad board)
At the start: 2 copper layers, 90 x 90 mm, 88 parts, among them CON1 SheldArduino, J1 Conn_01x02_Female, J10 DIGITAL, J11 DIGITAL, J12 Alimentacion, J13 Conn_01x02_Female, J2 3V3, J3 Conn_01x02_Female, J4 12V, J5 IN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

Commit message: Actualizacion
Parts:
- R15: moved to B.Cu
- moved R15 16.5 mm to (62.9, 83.1)
Routing:
- net GND: track 0.00 -> 338.2 mm
- net +5V: track 0.00 -> 255.0 mm
- net SCL: track 0.00 -> 196.0 mm
- net SDA: track 0.00 -> 194.5 mm
- net D12: track 0.00 -> 157.1 mm
- net RX: track 0.00 -> 151.8 mm
- net TX: track 0.00 -> 149.3 mm, vias 0 -> 1
- net PWM11: track 0.00 -> 102.8 mm
- net AIN0: track 0.00 -> 98.1 mm
- net D13: track 0.00 -> 92.4 mm
- net PWM6: track 0.00 -> 91.6 mm
- net RST: track 0.00 -> 89.0 mm
- net PWM10: track 0.00 -> 87.8 mm
- net AREF: track 0.00 -> 84.6 mm
- net PWM5: track 0.00 -> 77.3 mm
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Other:
- outline, holes or cut-outs redrawn
